Commit message: Added IKFast plugin. IK requests still failing

File: abb_irb1200_support/urdf/irb1200.urdf (robot description, URDF)
Before this commit: robot abb_irb1200, 9 links, 8 joints
Joints:
- joint joint_1: limit lower=-3.1416 upper=3.1416 effort=0 velocity=2.618 -> lower=-2.96705973 upper=2.96705973 effort=0 velocity=5.0265; origin xyz=0 0 0 rpy=0 0 0 -> xyz=0 0 0.219 rpy=0 0 0
- joint joint_2: limit lower=-1.7453 upper=1.9199 effort=0 velocity=2.618 -> lower=-1.74533 upper=2.35619 effort=0 velocity=4.18879; origin xyz=0.1 0 0.615 rpy=0 0 0 -> xyz=0 0 0.1801 rpy=0 0 0
- joint joint_3: limit lower=-1.0472 upper=1.1345 effort=0 velocity=2.618 -> lower=-3.49066 upper=1.22173 effort=0 velocity=5.2360; origin xyz=0 0 0.705 rpy=0 0 0 -> xyz=0 0 0.35 rpy=0 0 0
- joint joint_4: limit lower=-3.49 upper=3.49 effort=0 velocity=6.2832 -> lower=-4.71239 upper=4.71239 effort=0 velocity=6.98131; origin xyz=0.258 0 0.135 rpy=0 0 0 -> xyz=0.1885 0 0.042 rpy=0 0 0
- joint joint_5: limit lower=-2.0944 upper=2.0944 effort=0 velocity=6.2832 -> lower=-2.26893 upper=2.26893 effort=0 velocity=7.0686; origin xyz=0.497 0 0 rpy=0 0 0 -> xyz=0.1555 0 0 rpy=0 0 0
- joint joint_6: limit lower=-6.9813 upper=6.9813 effort=0 velocity=7.854 -> lower=-6.2832 upper=6.2832 effort=0 velocity=10.4720; origin xyz=0.085 0 0 rpy=0 0 0 -> xyz=0.077 0 0 rpy=0 0 0
