Commit message: Added end effector to robot. Not correctly lined up but good enough for demo.

File: abb_irb1200_support/urdf/irb1200_macro.xacro (robot description, xacro)
@@ -136,5 +136,24 @@
         </collision>
     </link>
-    <link name="${prefix}tool0"/>
+    <link name="${prefix}tool0">
+        <visual>
+            <origin xyz="
+                0 0.077 0.068" rpy="0 3.14159 -1.571"/>
+            <!-- <origin xyz=" -->
+                <!-- -${link_6_X+link_5_X+link_4_X+link_3_X+link_2_X+link_1_X} -${link_6_Y+link_5_Y+link_4_Y+link_3_Y+link_2_Y+link_1_Y} -${link_6_Z+link_5_Z+link_4_Z+link_3_Z+link_2_Z+link_1_Z}" rpy="0 0 0"/> -->
+            <geometry>
+                <mesh filename="package://abb_irb1200_support/meshes/irb1200/visual/ee.stl" scale="0.001 0.001 0.001"/>
+            </geometry>
+            <material name="abb_orange"/>
+        </visual>
+        <collision>
+            <origin xyz="
+                -${link_6_X+link_5_X+link_4_X+link_3_X+link_2_X+link_1_X} -${link_6_Y+link_5_Y+link_4_Y+link_3_Y+link_2_Y+link_1_Y} -${link_6_Z+link_5_Z+link_4_Z+link_3_Z+link_2_Z+link_1_Z}" rpy="0 0 0"/>
+            <geometry>
+                <mesh filename="package://abb_irb1200_support/meshes/irb1200/collision/ee.stl"  scale="0.001 0.001 0.001"/>
+            </geometry>
+            <material name="yellow"/>
+        </collision>
+    </link>
     <!-- end of link list -->
     <!-- joint list -->

Commit message: Added updates to preliminary adding of ee to model

File: abb_irb1200_support/urdf/irb1200_macro.xacro (robot description, xacro)
@@ -143,5 +143,5 @@
                 <!-- -${link_6_X+link_5_X+link_4_X+link_3_X+link_2_X+link_1_X} -${link_6_Y+link_5_Y+link_4_Y+link_3_Y+link_2_Y+link_1_Y} -${link_6_Z+link_5_Z+link_4_Z+link_3_Z+link_2_Z+link_1_Z}" rpy="0 0 0"/> -->
             <geometry>
-                <mesh filename="package://abb_irb1200_support/meshes/irb1200/visual/ee.stl" scale="0.001 0.001 0.001"/>
+                <mesh filename="package://abb_irb1200_support/meshes/irb1200/visual/ee_subsampled.stl" scale="0.001 0.001 0.001"/>
             </geometry>
             <material name="abb_orange"/>
@@ -151,5 +151,5 @@
                 -${link_6_X+link_5_X+link_4_X+link_3_X+link_2_X+link_1_X} -${link_6_Y+link_5_Y+link_4_Y+link_3_Y+link_2_Y+link_1_Y} -${link_6_Z+link_5_Z+link_4_Z+link_3_Z+link_2_Z+link_1_Z}" rpy="0 0 0"/>
             <geometry>
-                <mesh filename="package://abb_irb1200_support/meshes/irb1200/collision/ee.stl"  scale="0.001 0.001 0.001"/>
+                <mesh filename="package://abb_irb1200_support/meshes/irb1200/collision/ee_subsampled.stl"  scale="0.001 0.001 0.001"/>
             </geometry>
             <material name="yellow"/>

Commit message: added new extruder stl along with the collision stl, and updated urdf.

File: abb_irb1200_support/urdf/irb1200_macro.xacro (robot description, xacro)
@@ -136,12 +136,13 @@
         </collision>
     </link>
-    <link name="${prefix}tool0">
-        <visual>
-            <origin xyz="
-                0 0.077 0.068" rpy="0 3.14159 -1.571"/>
+    <link name="${prefix}tool0"/>
+    <link name="${prefix}extruder">
+        <visual>
+            <origin xyz="
+                0 0 .00875" rpy="0 3.14159 -1.571"/>
             <!-- <origin xyz=" -->
                 <!-- -${link_6_X+link_5_X+link_4_X+link_3_X+link_2_X+link_1_X} -${link_6_Y+link_5_Y+link_4_Y+link_3_Y+link_2_Y+link_1_Y} -${link_6_Z+link_5_Z+link_4_Z+link_3_Z+link_2_Z+link_1_Z}" rpy="0 0 0"/> -->
             <geometry>
-                <mesh filename="package://abb_irb1200_support/meshes/irb1200/visual/ee_subsampled.stl" scale="0.001 0.001 0.001"/>
+                <mesh filename="package://abb_irb1200_support/meshes/irb1200/visual/extruder.stl" scale="0.001 0.001 0.001"/>
             </geometry>
             <material name="abb_orange"/>
@@ -151,5 +152,5 @@
                 -${link_6_X+link_5_X+link_4_X+link_3_X+link_2_X+link_1_X} -${link_6_Y+link_5_Y+link_4_Y+link_3_Y+link_2_Y+link_1_Y} -${link_6_Z+link_5_Z+link_4_Z+link_3_Z+link_2_Z+link_1_Z}" rpy="0 0 0"/>
             <geometry>
-                <mesh filename="package://abb_irb1200_support/meshes/irb1200/collision/ee_subsampled.stl"  scale="0.001 0.001 0.001"/>
+                <mesh filename="package://abb_irb1200_support/meshes/irb1200/collision/extruder_collision.stl"  scale="0.001 0.001 0.001"/>
             </geometry>
             <material name="yellow"/>
@@ -205,4 +206,9 @@
         <origin xyz="0 0 0" rpy="0 1.57079632679 0"/>
     </joint>
+    <joint name="${prefix}joint_6-tool0-extruder" type="fixed">
+        <parent link="${prefix}tool0"/>
+        <child link="${prefix}extruder"/>
+        <origin xyz="0 0 0" rpy="0 0 0"/>
+    </joint>
     <!-- end of joint list -->
     <!-- ROS base_link to ABB World Coordinates transform -->

Commit message: end of extruder is now joint "extruder tip"

File: abb_irb1200_support/urdf/irb1200_macro.xacro (robot description, xacro)
@@ -137,5 +137,5 @@
     </link>
     <link name="${prefix}tool0"/>
-    <link name="${prefix}extruder">
+    <link name="${prefix}extruder_base">
         <visual>
             <origin xyz="
@@ -157,4 +157,5 @@
         </collision>
     </link>
+    <link name="${prefix}extruder_tip"/>
     <!-- end of link list -->
     <!-- joint list -->
@@ -206,8 +207,13 @@
         <origin xyz="0 0 0" rpy="0 1.57079632679 0"/>
     </joint>
-    <joint name="${prefix}joint_6-tool0-extruder" type="fixed">
+    <joint name="${prefix}tool0-extruder" type="fixed">
         <parent link="${prefix}tool0"/>
-        <child link="${prefix}extruder"/>
+        <child link="${prefix}extruder_base"/>
         <origin xyz="0 0 0" rpy="0 0 0"/>
+    </joint>
+    <joint name="${prefix}extruder_tip" type="fixed">
+        <parent link="${prefix}extruder_base"/>
+        <child link="${prefix}extruder_tip"/>
+        <origin xyz="0 0.0825 0.166525" rpy="0 0 0"/>
     </joint>
     <!-- end of joint list -->

Commit message: rotated extruder 90 deg

File: abb_irb1200_support/urdf/irb1200_macro.xacro (robot description, xacro)
@@ -140,5 +140,5 @@
         <visual>
             <origin xyz="
-                0 0 .00875" rpy="0 3.14159 -1.571"/>
+                0 0 .00875" rpy="0 3.14159 3.14159"/>
             <!-- <origin xyz=" -->
                 <!-- -${link_6_X+link_5_X+link_4_X+link_3_X+link_2_X+link_1_X} -${link_6_Y+link_5_Y+link_4_Y+link_3_Y+link_2_Y+link_1_Y} -${link_6_Z+link_5_Z+link_4_Z+link_3_Z+link_2_Z+link_1_Z}" rpy="0 0 0"/> -->
@@ -215,5 +215,5 @@
         <parent link="${prefix}extruder_base"/>
         <child link="${prefix}extruder_tip"/>
-        <origin xyz="0 0.0825 0.166525" rpy="0 0 0"/>
+        <origin xyz="0.0825 0 0.166525" rpy="0 0 0"/>
     </joint>
     <!-- end of joint list -->

Commit message: added collision quality stls of the robot.

File: abb_irb1200_support/urdf/irb1200_macro.xacro (robot description, xacro)
@@ -150,7 +150,7 @@
         <collision>
             <origin xyz="
-                -${link_6_X+link_5_X+link_4_X+link_3_X+link_2_X+link_1_X} -${link_6_Y+link_5_Y+link_4_Y+link_3_Y+link_2_Y+link_1_Y} -${link_6_Z+link_5_Z+link_4_Z+link_3_Z+link_2_Z+link_1_Z}" rpy="0 0 0"/>
-            <geometry>
-                <mesh filename="package://abb_irb1200_support/meshes/irb1200/collision/extruder_collision.stl"  scale="0.001 0.001 0.001"/>
+                0 0 .00875" rpy="0 3.14159 3.14159"/>
+            <geometry>
+                <mesh filename="package://abb_irb1200_support/meshes/irb1200/collision/extruder.stl"  scale="0.001 0.001 0.001"/>
             </geometry>
             <material name="yellow"/>

Commit message: Added bed (visual and collision) stls. still needs to be moved to the correct position.

File: abb_irb1200_support/urdf/irb1200_macro.xacro (robot description, xacro)
@@ -218,4 +218,26 @@
     </joint>
     <!-- end of joint list -->
+    <!-- enviroment list-->
+    <link name="build_platform">
+        <visual>
+            <origin xyz="0 0 0" rpy="0 0 0"/>
+            <geometry>
+                <mesh filename="package://abb_irb1200_support/meshes/buildplatform/visual/buildplatform.stl" scale="0.001 0.001 0.001"/>
+            </geometry>
+            <material name="abb_orange"/>
+        </visual>
+        <collision>
+            <geometry>
+                <mesh filename="package://abb_irb1200_support/meshes/buildplatform/collision/buildplatform.stl" scale="0.001 0.001 0.001"/>
+            </geometry>
+            <material name="yellow"/>
+        </collision>
+    </link>
+    <joint name="platform" type="fixed">
+        <parent link="${prefix}base_link"/>
+        <child link="build_platform"/>
+        <origin xyz="0.6 0 0" rpy="0 0 0"/>
+    </joint>
+    <!-- end enviroment list-->
     <!-- ROS base_link to ABB World Coordinates transform -->
     <link name="${prefix}base" />

Commit message: bed has been moved to the correct (approximate) position

File: abb_irb1200_support/urdf/irb1200_macro.xacro (robot description, xacro)
@@ -237,5 +237,5 @@
         <parent link="${prefix}base_link"/>
         <child link="build_platform"/>
-        <origin xyz="0.6 0 0" rpy="0 0 0"/>
+        <origin xyz="0.567 0 0" rpy="0 0 0"/>
     </joint>
     <!-- end enviroment list-->

Commit message: Changed cologrs on urdf

File: abb_irb1200_support/urdf/irb1200_macro.xacro (robot description, xacro)
@@ -9,6 +9,9 @@
                 <mesh filename="package://abb_irb1200_support/meshes/irb1200/visual/base_link.stl"/>
             </geometry>
-            <material name="abb_orange">
-                <color rgba="1 0.43 0 1"/>
+            <!-- <material name="abb_orange"> -->
+                <!-- <color rgba="1 0.43 0 1"/> -->
+            <!-- </material> -->
+            <material name="whitesmoke">
+                <color rgba="0.8 0.8 0.8 1"/>
             </material>
         </visual>
@@ -28,5 +31,5 @@
                 <mesh filename="package://abb_irb1200_support/meshes/irb1200/visual/link_1.stl"/>
             </geometry>
-            <material name="abb_orange"/>
+            <material name="whitesmoke"/>
         </visual>
         <collision>
@@ -47,5 +50,5 @@
                 <mesh filename="package://abb_irb1200_support/meshes/irb1200/visual/link_2.stl"/>
             </geometry>
-            <material name="abb_orange"/>
+            <material name="whitesmoke"/>
         </visual>
         <collision>
@@ -69,5 +72,5 @@
                 <mesh filename="package://abb_irb1200_support/meshes/irb1200/visual/link_3.stl"/>
             </geometry>
-            <material name="abb_orange"/>
+            <material name="whitesmoke"/>
         </visual>
         <collision>
@@ -89,5 +92,5 @@
                 <mesh filename="package://abb_irb1200_support/meshes/irb1200/visual/link_4.stl"/>
             </geometry>
-            <material name="abb_orange"/>
+            <material name="whitesmoke"/>
         </visual>
         <collision>
@@ -107,5 +110,5 @@
                 <mesh filename="package://abb_irb1200_support/meshes/irb1200/visual/link_5.stl"/>
             </geometry>
-            <material name="abb_orange"/>
+            <material name="whitesmoke"/>
         </visual>
         <collision>
@@ -125,5 +128,5 @@
                 <mesh filename="package://abb_irb1200_support/meshes/irb1200/visual/link_6.stl"/>
             </geometry>
-            <material name="abb_orange"/>
+            <material name="whitesmoke"/>
         </visual>
         <collision>
@@ -146,5 +149,7 @@
                 <mesh filename="package://abb_irb1200_support/meshes/irb1200/visual/extruder.stl" scale="0.001 0.001 0.001"/>
             </geometry>
-            <material name="abb_orange"/>
+            <material name="silver">
+                <color rgba="0.753 0.753 0.753 1"/>
+            </material>
         </visual>
         <collision>
@@ -225,5 +230,7 @@
                 <mesh filename="package://abb_irb1200_support/meshes/buildplatform/visual/buildplatform.stl" scale="0.001 0.001 0.001"/>
             </geometry>
-            <material name="abb_orange"/>
+            <material name="">
+                <color rgba="0.475 0.475 0.475 1"/>
+            </material>
         </visual>
         <collision>

Commit message: Added joint limits

File: abb_irb1200_support/urdf/irb1200_macro.xacro (robot description, xacro)
@@ -191,5 +191,6 @@
         <child link="${prefix}link_4"/>
         <axis xyz="1 0 0"/>
-        <limit lower="-4.71239" upper="4.71239" effort="0" velocity="6.98131"/>
+        <!-- <limit lower="-4.71239" upper="4.71239" effort="0" velocity="6.98131"--> <!-- this is the hard limits -->
+        <limit lower="-1.57079632679" upper="1.57079632679" effort="0" velocity="6.98131"/>
     </joint>
     <joint name="${prefix}joint_5" type="revolute">
@@ -205,5 +206,6 @@
         <child link="${prefix}link_6"/>
         <axis xyz="1 0 0"/>
-        <limit lower="-6.2832" upper="6.2832" effort="0" velocity="10.4720"/>
+        <!-- <limit lower="-6.2832" upper="6.2832" effort="0" velocity="10.4720"-->  <!-- this is the hard limits -->
+        <limit lower="0.78539816339" upper="2.35619449019" effort="0" velocity="10.4720"/>
     </joint>
     <joint name="${prefix}joint_6-tool0" type="fixed">

Commit message: Updated z height for machined extruder tip

File: abb_irb1200_support/urdf/irb1200_macro.xacro (robot description, xacro)
@@ -222,5 +222,5 @@
         <parent link="${prefix}extruder_base"/>
         <child link="${prefix}extruder_tip"/>
-        <origin xyz="0.0825 0 0.166525" rpy="0 0 0"/>
+        <origin xyz="0.0825 0 0.16533" rpy="0 0 0"/>
     </joint>
     <!-- end of joint list -->
